File: ENS_light_sw_board.kicad_sch (KiCad schematic)
At the start: 17 parts, among them J1 Conn_02x05_Odd_Even, SW1 SW_SPST, SW2 SW_SPST, SW3 SW_SPST, SW4 SW_SPST

Commit message: prod v1
Parts:
- SW1, SW2, SW3, SW4: footprint (none) -> Button_Switch_SMD:SW_Push_1P1T_XKB_TS-1187A
